Commit message: fix urdf translations

File: iplow_description/urdf/base.urdf.xacro (robot description, xacro)
@@ -11,4 +11,5 @@
     <link name="${name}">
 			<visual>
+        <origin xyz="0 0.0569 0.0" rpy="0 0 0"/>
 				<geometry>
 					<mesh filename="package://iplow_description/meshes/base.stl"/>
@@ -16,4 +17,5 @@
 			</visual>
 			<collision>
+        <origin xyz="0 0.0569 0.0" rpy="0 0 0"/>
 				<geometry>
 					<mesh filename="package://iplow_description/meshes/base.stl"/>

File: iplow_description/urdf/iplow_core.urdf.xacro (robot description, xacro)
@@ -2,5 +2,9 @@
 <robot xmlns:xacro="http://www.ros.org/wiki/xacro">
   <xacro:include filename="base.urdf.xacro"/>
+  <xacro:include filename="left_wheel.urdf.xacro"/>
   <xacro:include filename="right_wheel.urdf.xacro"/>
+  <xacro:include filename="left_caster.urdf.xacro"/>
+  <xacro:include filename="right_caster.urdf.xacro"/>
+  <xacro:include filename="mid360.urdf.xacro"/>
   <!-- <link name="world"> -->
   <!-- </link> -->
@@ -13,8 +17,26 @@
   <link name="base_link"/>
   <xacro:base name="base" parent="base_link">
-    <origin xyz="0 0 0.355" rpy="0 0 ${pi/2}"/> <!-- wheels touch the ground with z=0.345-->
+    <origin xyz="0 0 0.38" rpy="0 0 0"/> <!-- wheels touch the ground with z=0.3784-->
   </xacro:base>
-  <xacro:right_back_arm name="right_wheel" parent="base">
-    <origin xyz="0 0 0.355" rpy="0 0 ${pi/2}"/> <!-- wheels touch the ground with z=0.345-->
-  </xacro:right_back_arm>
+  <joint name="odom_joint" type="fixed">
+    <parent link="base"/>
+    <child link="odom"/>
+    <origin xyz="0 0 0" rpy="0 0 0"/>
+  </joint>
+  <link name="odom"/>
+  <xacro:left_wheel name="left_wheel" parent="base">
+    <origin xyz="-0.3129 0.0 -0.2234" rpy="0 0 0"/>
+  </xacro:left_wheel>
+  <xacro:right_wheel name="right_wheel" parent="base">
+    <origin xyz="0.3129 0.0 -0.2234" rpy="0 0 0"/>
+  </xacro:right_wheel>
+  <xacro:left_caster name="left_caster" parent="base">
+    <origin xyz="-0.3006 0.4594 -0.3152" rpy="0 0 0"/>
+  </xacro:left_caster>
+  <xacro:right_caster name="right_caster" parent="base">
+    <origin xyz="0.2951 0.471064 -0.3102" rpy="0 0 0"/>
+  </xacro:right_caster>
+  <xacro:mid360 name="mid360" parent="base">
+    <origin xyz="-0.002 -0.0632 0.9655" rpy="0 0 0"/>
+  </xacro:mid360>
 </robot>

File: iplow_description/urdf/right_wheel.urdf.xacro (robot description, xacro)
@@ -3,5 +3,5 @@
   <xacro:include filename="inertial_macros.urdf.xacro"/>
 	<xacro:arg name="ignition" default="false"/>
-	<xacro:macro name="right_back_arm" params="name parent *origin">
+	<xacro:macro name="right_wheel" params="name parent *origin">
     <joint name="${name}_joint" type="continuous">
 			<parent link="${parent}"/>
